File: nfc_card.kicad_sch (KiCad schematic)
At the start: 5 parts, among them IC1 NT3H2111W0FHKH

Commit message: Start schematic
Parts:
- D1: footprint (none) -> LED_SMD:LED_0805_2012Metric
- IC1: footprint QFN50P160X160X50-8N -> NT3H2111W0FHKH:QFN50P160X160X50-8N
- R1: footprint (none) -> Resistor_SMD:R_0402_1005Metric
Changed lines of the file:
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@@
 			)
 		)
-		(property "Footprint" ""
+		(property "Footprint" "Resistor_SMD:R_0402_1005Metric"
 			(at 68.58 105.41 0)
 			(effects
@@
 			)
 		)
-		(property "Footprint" ""
+		(property "Footprint" "LED_SMD:LED_0805_2012Metric"
 			(at 59.69 105.41 0)
 			(effects
@@
 			)
 		)
-		(property "Footprint" "QFN50P160X160X50-8N"
+		(property "Footprint" "NT3H2111W0FHKH:QFN50P160X160X50-8N"
 			(at 76.2 160.96 0)
 			(effects

Commit message: Add antenna
Parts:
- AE1: value Antenna_Loop -> 25x48mm; footprint (none) -> NFC:Antenna_25x48mm
Connections:
- net ANT1: now reaches AE1.1, IC1.1 (LA)
- net ANT2: now reaches AE1.2, IC1.8 (LB)
Changed lines of the file:
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@@
+		)
+	)
+	(label "ANT1"
+		(at 46.99 63.5 90)
+		(fields_autoplaced yes)
+		(effects
+			(font
+				(size 1.27 1.27)
+			)
+			(justify left bottom)
+		)
+	)
+	(label "ANT2"
+		(at 55.88 55.88 0)
+		(fields_autoplaced yes)
+		(effects
+			(font
+				(size 1.27 1.27)
+			)
+			(justify left bottom)
 		)
 	)
@@
 			)
 		)
-		(property "Value" "Antenna_Loop"
+		(property "Value" "25x48mm"
 			(at 53.34 46.9899 0)
 			(effects
@@
 			)
 		)
-		(property "Footprint" ""
+		(property "Footprint" "NFC:Antenna_25x48mm"
 			(at 46.99 45.72 0)
 			(effects
